File: clock_pcb/2.kicad_sch (KiCad schematic)
At the start: 69 parts, among them J1 USB_C_Receptacle_USB2.0, J2 PROG, Q1 AO3401A, Q2 AO3401A, SW1 TS-1187A-B-A-B, SW2 SSSS811101, SW3 TS-1187A-B-A-B, U1 RP2040, U2 SRV05-4, U3 RT9080-33GJ5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

Commit message: finished schematic parts, layout outline
Parts:
- renumbered R2 to R1, R9 to R10, R12 to R11, R11 to R12, R16 to R15, R17 to R16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
Connections:
- net USB_D+: now also U1.3 (IO2); no longer U1.1 (IO1)
- net USB_D-: now also U1.1 (IO1); no longer U1.3 (IO2)
