File: clock_pcb/PAGE2.kicad_sch (KiCad schematic)
At the start: 69 parts, among them J1 USB_C_Receptacle_USB2.0, J2 PROG, Q1 AO3401A, Q2 AO3401A, SW1 TS-1187A-B-A-B, SW2 SSSS811101, SW3 TS-1187A-B-A-B, U1 RP2040, U2 SRV05-4, U3 RT9080-33GJ5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

Commit message: changed all to single sided
Parts:
- J1: lcsc C167321 -> C2843970
Changed lines of the file:
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@@
       (effects (font (size 1.27 1.27)) hide)
     )
-    (property "lcsc" "C167321" (at 27.94 40.005 0)
+    (property "lcsc" "C2843970" (at 27.94 40.005 0)
       (effects (font (size 1.27 1.27)) hide)
     )
@@
       (effects (font (size 1.27 1.27)) hide)
     )
+    (property "digi" "" (at 27.94 40.005 0)
+      (effects (font (size 1.27 1.27)) hide)
+    )

Commit message: layout work
Parts:
- removed TP2: GND, TestPoint:TestPoint_Pad_D1.0mm, symbol Connector:TestPoint_Small
- removed TP6, TP8: 5V, TestPoint:TestPoint_Pad_D1.0mm, symbol Connector:TestPoint_Small
- SW2: renamed from SW1; footprint Button_Switch_SMD:SW_SPST_TL3342 -> stride_footprints:SW_SPST_TL3342_RT
- SW3: footprint Button_Switch_SMD:SW_SPST_TL3342 -> stride_footprints:SW_SPST_TL3342_RT
- renumbered SW2 to SW1
Connections:
- net USB_D+: now also U2.3 (IO2); no longer U2.1 (IO1)
- net USB_D-: now also U2.1 (IO1); no longer U2.3 (IO2)
