File: clock_pcb/PAGE3.kicad_sch (KiCad schematic)
At the start: 43 parts, among them J3 FFC 24, J4 5V, J5 5V, J6 OLED, J7 5V, J8 5V, Q3 2N7002, Q5 AO3400A, SW4 TS-1187A-B-A-B, SW5 TS-1187A-B-A-B, U5 DS1307Z+, Y2 32.768kHz

Commit message: finished schematic parts, layout outline
Parts:
- removed J8: 5V, Connector_JST:JST_SH_SM02B-SRSS-TB_1x02-1MP_P1.00mm_Horizontal, symbol Connector_Generic:Conn_01x02
- added BZ1: CMT-8504-100-SMT-TR, Buzzer_Beeper:MagneticBuzzer_CUI_CMT-8504-100-SMT, symbol stride_symbols:Buzzer_CMT-8504-100-SMT-TR
- BT1: footprint ftp:Q&J_CR2032-BS-6-1 -> stride_footprints:Q&J_CR2032-BS-6-1
- D5: footprint ftp:WS2812B-2020 -> stride_footprints:WS2812B-2020
- J7: renamed from J6; footprint ftp:OLED-128O064D_edit -> stride_footprints:OLED-128O064D_edit_reverse_v2
- renumbered C1 to C22, C22 to C23, C23 to C24, C24 to C25, C25 to C27, C27 to C28, C28 to C29, C29 to C30, C30 to C32, J7 to J4, J4 to J6, Q5 to Q3, Q3 to Q4, R32 to R19, R19 to R20, R31 to R21, R20 to R22, R22 to R23, R21 to R24, R23 to R25, R25 to R26, R24 to R27, R26 to R28, R27 to R29, R28 to R30, R29 to R31
Connections:
- net BUZZER_HIGH: now also BZ1.1 (-)
- net BUZZER_LOW: now also D6.2 (A), BZ1.2 (+), BZ1.3 (DUMMY1), BZ1.4 (DUMMY2)
- net GND: no longer D6.2 (A)
Other:
- note removed: "Piezo long pin usually (+)"
- moved on the sheet: C22, Q3, R19, R21

Commit message: layout work
Parts:
- added C33: 1u, Capacitor_SMD:C_0402_1005Metric, symbol Device:C_Small
- SW4, SW5: footprint Button_Switch_SMD:SW_SPST_TL3342 -> stride_footprints:SW_SPST_TL3342_RT
Connections:
- net +3V3: now also C33.1
- net GND: now also C33.2
- net WS2812_RGB_LED renamed GPIO13_WS2812_RGB_LED
Changed lines of the file:
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@@
   (junction (at 242.57 85.09) (diameter 0) (color 0 0 0 0)
   )
-  (junction (at 259.08 148.59) (diameter 0) (color 0 0 0 0)
+  (junction (at 228.6 57.15) (diameter 0) (color 0 0 0 0)
   )
-  (junction (at 228.6 46.99) (diameter 0) (color 0 0 0 0)
+  (junction (at 259.08 148.59) (diameter 0) (color 0 0 0 0)
   )
   (junction (at 177.292 127.381) (diameter 0) (color 0 0 0 0)
@@
   (junction (at 242.57 67.31) (diameter 0) (color 0 0 0 0)
   )
+  (junction (at 228.6 46.99) (diameter 0) (color 0 0 0 0)
+  )
   (junction (at 262.89 46.99) (diameter 0) (color 0 0 0 0)
   )
@@
   (junction (at 242.57 77.47) (diameter 0) (color 0 0 0 0)
   )
+  (junction (at 222.25 46.99) (diameter 0) (color 0 0 0 0)
+  )
   (junction (at 252.095 148.59) (diameter 0) (color 0 0 0 0)
   )
@@
   )
   (no_connect (at 265.43 41.91))
+  (wire (pts (xy 228.6 57.15) (xy 235.585 57.15))
+    (stroke (width 0) (type default))
+  )
   (wire (pts (xy 139.7 170.18) (xy 118.745 170.18))
     (stroke (width 0) (type default))
   )
+  (wire (pts (xy 222.25 46.99) (xy 228.6 46.99))
+    (stroke (width 0) (type default))
+  )
   (wire (pts (xy 127.762 137.541) (xy 109.982 137.541))
     (stroke (width 0) (type default))
@@
     (stroke (width 0) (type default))
   )
-  (wire (pts (xy 228.6 44.45) (xy 228.6 46.99))
-    (stroke (width 0) (type default))
-  )
   (wire (pts (xy 137.795 41.91) (xy 143.51 41.91))
     (stroke (width 0) (type default))
@@
     (stroke (width 0) (type default))
   )
+  (wire (pts (xy 222.25 53.975) (xy 222.25 57.15))
+    (stroke (width 0) (type default))
+  )
   (wire (pts (xy 162.56 44.45) (xy 162.56 42.545))
     (stroke (width 0) (type default))
@@
     (stroke (width 0) (type default))
   )
-  (wire (pts (xy 228.6 57.15) (xy 235.585 57.15))
+  (wire (pts (xy 222.25 57.15) (xy 228.6 57.15))
     (stroke (width 0) (type default))
   )
@@
     (stroke (width 0) (type default))
   )
+  (wire (pts (xy 222.25 44.45) (xy 222.25 46.99))
+    (stroke (width 0) (type default))
+  )
   (wire (pts (xy 175.895 51.435) (xy 175.895 52.705))
     (stroke (width 0) (type default))
@@
     (stroke (width 0) (type default))
   )
+  (wire (pts (xy 222.25 46.99) (xy 222.25 48.895))
+    (stroke (width 0) (type default))
+  )
   (wire (pts (xy 185.42 83.82) (xy 185.42 86.36))
     (stroke (width 0) (type solid))
@@
     (effects (font (size 1.27 1.27)) (justify right bottom))
   )
-  (global_label "WS2812_RGB_LED" (shape input) (at 181.102 137.541 0) (fields_autoplaced)
+  (global_label "GPIO13_WS2812_RGB_LED" (shape input) (at 181.102 137.541 0) (fields_autoplaced)
     (effects (font (size 1 1)) (justify left))
-    (property "Intersheetrefs" "${INTERSHEET_REFS}" (at 196.1449 137.4785 0)
+    (property "Intersheetrefs" "${INTERSHEET_REFS}" (at 202.7234 137.541 0)
       (effects (font (size 1 1)) (justify left) hide)
     )
@@
     )
   )
-  (symbol (lib_id "power:+3V3") (at 228.6 44.45 0) (unit 1)
-    (in_bom yes) (on_board yes) (dnp no)
-    (property "Reference" "#PWR071" (at 228.6 48.26 0)
-      (effects (font (size 1.27 1.27)) hide)
-    )
-    (property "Value" "+3V3" (at 228.6 40.64 0)
-      (effects (font (size 1.27 1.27)))
-    )
-    (property "Footprint" "" (at 228.6 44.45 0)
-      (effects (font (size 1.27 1.27)) hide)
-    )
-    (property "Datasheet" "" (at 228.6 44.45 0)
-      (effects (font (size 1.27 1.27)) hide)
-    )
-    (pin "1")
-    (instances
-      (project "clock_pcb"
-        (path "/e63e39d7-6ac0-4ffd-8aa3-1841a4541b55/05d988ef-d5db-40c4-a11a-450249f6a23d"
-          (reference "#PWR071") (unit 1)
-        )
-      )
-    )
-  )
   (symbol (lib_id "Device:Battery_Cell") (at 161.925 78.74 0) (unit 1)
     (in_bom yes) (on_board yes) (dnp no) (fields_autoplaced)
@@
       (effects (font (size 1.27 1.27)) hide)
     )
-    (property "Footprint" "Button_Switch_SMD:SW_SPST_TL3342" (at 157.48 49.53 0)
+    (property "Footprint" "stride_footprints:SW_SPST_TL3342_RT" (at 157.48 49.53 0)
       (effects (font (size 1.27 1.27)) hide)
     )
@@
       (effects (font (size 1.27 1.27)) hide)
     )
+    (property "digi" "" (at 162.56 49.53 0)
+      (effects (font (size 1.27 1.27)) hide)
+    )
+    (property "bom" "" (at 162.56 49.53 0)
+      (effects (font (size 1.27 1.27)) hide)
+    )
     (pin "1")
     (pin "2")
@@
       (effects (font (size 1.27 1.27)) hide)
     )
-    (property "Footprint" "Button_Switch_SMD:SW_SPST_TL3342" (at 125.095 48.895 0)
+    (property "Footprint" "stride_footprints:SW_SPST_TL3342_RT" (at 125.095 48.895 0)
       (effects (font (size 1.27 1.27)) hide)
     )
@@
       (effects (font (size 1.27 1.27)) hide)
     )
+    (property "digi" "" (at 130.175 48.895 0)
+      (effects (font (size 1.27 1.27)) hide)
+    )
+    (property "bom" "" (at 130.175 48.895 0)
+      (effects (font (size 1.27 1.27)) hide)
+    )
     (pin "1")
     (pin "2")
@@
     )
   )
+  (symbol (lib_id "Device:C_Small") (at 222.25 51.435 0) (unit 1)
+    (in_bom yes) (on_board yes) (dnp no)
+    (property "Reference" "C33" (at 223.52 49.53 0)
+      (effects (font (size 1.27 1.27)) (justify left))
+    )
+    (property "Value" "1u" (at 224.155 53.975 0)
+      (effects (font (size 1.27 1.27)) (justify left))
+    )
+    (property "Footprint" "Capacitor_SMD:C_0402_1005Metric" (at 222.25 51.435 0)
+      (effects (font (size 1.27 1.27)) hide)
+    )
+    (property "Datasheet" "~" (at 222.25 51.435 0)
+      (effects (font (size 1.27 1.27)) hide)
+    )
+    (property "lcsc" "C52923" (at 222.25 51.435 0)
+      (effects (font (size 1.27 1.27)) hide)
+    )
+    (property "desc" "25V X5R" (at 222.25 51.435 0)
+      (effects (font (size 1.27 1.27)) hide)
+    )
+    (pin "1")
+    (pin "2")
+    (instances
+      (project "clock_pcb"
+        (path "/e63e39d7-6ac0-4ffd-8aa3-1841a4541b55/05d988ef-d5db-40c4-a11a-450249f6a23d"
+          (reference "C33") (unit 1)
+        )
+      )
+    )
+  )
   (symbol (lib_id "power:GND") (at 161.925 82.55 0) (mirror y) (unit 1)
     (in_bom yes) (on_board yes) (dnp no)
@@
         )
       )
+    )
+  )
+  (symbol (lib_id "power:+3V3") (at 222.25 44.45 0) (unit 1)
+    (in_bom yes) (on_board yes) (dnp no)
+    (property "Reference" "#PWR071" (at 222.25 48.26 0)
+      (effects (font (size 1.27 1.27)) hide)
+    )
+    (property "Value" "+3V3" (at 222.25 40.64 0)
+      (effects (font (size 1.27 1.27)))
+    )
+    (property "Footprint" "" (at 222.25 44.45 0)
+      (effects (font (size 1.27 1.27)) hide)
+    )
+    (property "Datasheet" "" (at 222.25 44.45 0)
+      (effects (font (size 1.27 1.27)) hide)
+    )
+    (pin "1")
+    (instances
+      (project "clock_pcb"
+        (path "/e63e39d7-6ac0-4ffd-8aa3-1841a4541b55/05d988ef-d5db-40c4-a11a-450249f6a23d"
+          (reference "#PWR071") (unit 1)
+        )
+      )
