File: clock_pcb/clock_pcb.kicad_pcb (KiCad board)
At the start: 2 copper layers, 100 x 50 mm, 107 parts, among them J1 USB_C_Receptacle_USB2.0, J2 PROG, J3 FFC 24, J4 5V, J5 5V, J6 OLED, J7 5V, J8 5V, Q1 AO3401A, Q2 AO3401A, Q3 2N7002, Q5 AO3400A, SW1 TS-1187A-B-A-B, SW2 SSSS811101, SW3 TS-1187A-B-A-B, SW4 TS-1187A-B-A-B, SW5 TS-1187A-B-A-B, U1 SRV05-4, U2 RP2040, U3 RT9080-33GJ5, U4 W25Q64JV, U5 DS1307Z+, Y1 XYDBPCNANF-12MHZ, Y2 32.768kHz

Commit message: finished schematic parts, layout outline
Parts:
- removed J8: 5V, Connector_JST:JST_SH_SM02B-SRSS-TB_1x02-1MP_P1.00mm_Horizontal
- removed Q5: AO3400A, Package_TO_SOT_SMD:SOT-23
- removed R32: 120, Resistor_SMD:R_0402_1005Metric
- added BZ1: CMT-8504-100-SMT-TR, Buzzer_Beeper:MagneticBuzzer_CUI_CMT-8504-100-SMT, F.Cu at (113.7, 141.2)
- added FID1: Fiducial, Fiducial:Fiducial_1mm_Mask2mm, F.Cu at (146.1, 156.5)
- added FID2: Fiducial, Fiducial:Fiducial_1mm_Mask2mm, F.Cu at (146.1, 160.1)
- added G***: LOGO, silk:subtitle, B.Cu at (65.0, 132.6)
- added G***: LOGO, silk:title, B.Cu at (69.8, 132.8)
- added G***: LOGO, silk:comb, B.Cu at (125.8, 107.7)
- added G***: LOGO, silk:flower, B.Cu at (84.5, 116.3)
- added G***: LOGO, silk:hummingbird, B.Cu at (104.4, 129.7)
- added G***: LOGO, silk:comb, B.Cu at (58.1, 110.6)
- added G***: LOGO, silk:comb, B.Cu at (143.4, 105.9)
- added H1: Tooling_Hole_JLC, stride_footprints:JLC_Tooling_Hole, F.Cu at (148.9, 155.8)
- added H2: Tooling_Hole_JLC, stride_footprints:JLC_Tooling_Hole, F.Cu at (148.9, 158.0)
- added H3: Tooling_Hole_JLC, stride_footprints:JLC_Tooling_Hole, F.Cu at (148.9, 160.1)
- added Q4: 2N7002, Package_TO_SOT_SMD:SOT-23, F.Cu at (29.3, 165.9)
- added R30: 1k, Resistor_SMD:R_0402_1005Metric, F.Cu at (151.4, 160.2)
- BT1: footprint ftp:Q&J_CR2032-BS-6-1 -> stride_footprints:Q&J_CR2032-BS-6-1
- C22: value 0.1u -> 10u
- C23, C25: value 1u -> 0.1u
- C24, C30: value 0.1u -> 1u
- C27: value 2.2u -> 1u
- C28: value 1u -> 2.2u
- C32: value 10u -> 0.1u
- D5: footprint ftp:WS2812B-2020 -> stride_footprints:WS2812B-2020
- J1: footprint ftp:USB-C-16p -> stride_footprints:USB-C-16p_vertical_GT-USB-7051A; moved to B.Cu
- J6: value OLED -> 5V; footprint Mitch_Library:OLED-128O064D_edit_reverse -> Connector_JST:JST_SH_SM02B-SRSS-TB_1x02-1MP_P1.00mm_Horizontal; moved to F.Cu
- J7: value 5V -> OLED; footprint Connector_JST:JST_SH_SM02B-SRSS-TB_1x02-1MP_P1.00mm_Horizontal -> stride_footprints:OLED-128O064D_edit_reverse_v2
- Q3: value 2N7002 -> AO3400A
- R1: value 5.1k -> 1k
- R10: value 10k -> 100k
- R11: value 2.2k -> 1k
- R12: value 1k -> 2.2k
- R15: value 0 -> 300; footprint master_ftp:R_0402_1005Metric_3pad -> Resistor_SMD:R_0402_1005Metric
- R16: footprint master_ftp:R_0402_1005Metric_3pad -> stride_footprints:R_0402_1005Metric_3pad
- R17: value 300 -> 0; footprint Resistor_SMD:R_0402_1005Metric -> stride_footprints:R_0402_1005Metric_3pad
- R19: value 10k -> 120
- R20: value 51 -> 10k
- R21, R28: value 1k -> 10k
- R22: value 10k -> 51
- R24: value 10k -> 1k
- R29: value 330k -> 10k
- R3: value 1k -> 5.1k
- R31: value 10k -> 330k
- R9: value 100k -> 10k
- SW2: footprint ftp:SSSS811101 -> stride_footprints:SSSS811101
- SW4, SW5: moved to B.Cu
- TP4: value 5V -> GND CLIP; footprint TestPoint:TestPoint_Pad_D1.0mm -> stride_footprints:ronghe_RH-5016_C5199799
- TP6: value 3V3 -> 5V
- TP7: value 5V -> 3V3
- TP8: value GND CLIP -> 5V; footprint Mitch_Library:ronghe_RH-5016_C5199799 -> TestPoint:TestPoint_Pad_D1.0mm
- U1: value SRV05-4 -> RP2040; footprint Package_TO_SOT_SMD:SOT-23-6 -> stride_footprints:QFN-56_EP_7x7_Pitch0.4mm
- U2: value RP2040 -> SRV05-4; footprint ftp:QFN-56_EP_7x7_Pitch0.4mm -> Package_TO_SOT_SMD:SOT-23-6
- moved C19 157.8 mm to (20.2, 185.3), turned to 90 degrees
- moved R18 156.3 mm to (21.4, 185.3), turned to -90 degrees
- moved R19 154.7 mm to (22.6, 185.3), turned to -90 degrees
- moved TP2 140.6 mm to (34.0, 164.8)
- moved J5 130.1 mm to (71.2, 104.6)
- moved J4 126.6 mm to (62.0, 104.2)
- moved D3 120.6 mm to (23.2, 130.0)
- moved SW5 120.5 mm to (56.1, 137.5)
- moved SW4 118.8 mm to (56.1, 130.0), turned to 0 degrees
- moved J1 113.3 mm to (60.0, 145.0), turned to 180 degrees
- moved F1 111.9 mm to (56.2, 145.0), turned to 90 degrees
- moved D2 109.9 mm to (29.3, 118.5)
- moved R8 109.9 mm to (32.9, 122.5)
- moved Q2 109.9 mm to (25.5, 119.2)
- moved R10 109.9 mm to (19.2, 119.8)
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Connections:
- net /PAGE3/WS2812_DOUT renamed /CONNS & PERIPHERALS/WS2812_DOUT
- C10 pad 1: Net-(U2-VREG_VOUT) -> Net-(U1-VREG_VOUT)
- C12 pad 2: Net-(U2-XIN) -> Net-(U1-XIN)
- C13 pad 2: Net-(U2-XOUT) -> Net-(U1-XOUT)
- C14 pad 1: Net-(U2-VREG_VOUT) -> Net-(U1-VREG_VOUT)
- C22 pad 1: BUTTON_1 -> /CONNS & PERIPHERALS/BUZZER_HIGH
- C23 pad 1: +3V3 -> BUTTON_1
- C24 pad 1: /PAGE3/OLED_RST -> +3V3
- C25 pad 1: +3V3 -> /CONNS & PERIPHERALS/OLED_RST
- C27 pad 1: GND -> +3V3
- C27 pad 2: Net-(J6-Pin_27) -> GND
- C28 pad 1: Net-(J6-Pin_3) -> GND
- C28 pad 2: Net-(J6-Pin_2) -> Net-(J7-Pin_27)
- C29 pad 1: Net-(J6-Pin_5) -> Net-(J7-Pin_3)
- C29 pad 2: Net-(J6-Pin_4) -> Net-(J7-Pin_2)
- C30 pad 1: GPIO26_ADC0_LDR -> Net-(J7-Pin_5)
- C30 pad 2: GND -> Net-(J7-Pin_4)
- C31 pad 2: Net-(J6-Pin_28) -> Net-(J7-Pin_28)
- C32 pad 1: /PAGE3/BUZZER_HIGH -> GPIO26_ADC0_LDR
- C5 pad 1: /PAGE2/~{RESET} -> /RP2040 & USB/~{RESET}
- C8 pad 1: Net-(U2-VREG_VOUT) -> Net-(U1-VREG_VOUT)
- D6 pad 1: /PAGE3/BUZZER_HIGH -> /CONNS & PERIPHERALS/BUZZER_HIGH
- D6 pad 2: GND -> /CONNS & PERIPHERALS/BUZZER_LOW
- J1 pad A6: /PAGE2/USB_D+ -> /RP2040 & USB/USB_D+
- J1 pad A7: /PAGE2/USB_D- -> /RP2040 & USB/USB_D-
- J1 pad B6: /PAGE2/USB_D+ -> /RP2040 & USB/USB_D+
- J1 pad B7: /PAGE2/USB_D- -> /RP2040 & USB/USB_D-
- J2 pad 1: /PAGE2/PROG1 -> /RP2040 & USB/PROG1
- J2 pad 3: /PAGE2/UART0_TX -> /RP2040 & USB/UART0_TX
- J2 pad 5: /PAGE2/UART0_RX -> /RP2040 & USB/UART0_RX
- J2 pad 6: /PAGE2/PROG2 -> /RP2040 & USB/PROG2
- J4 pad 1: GPIO26_ADC0_LDR -> GND
- J4 pad 2: Net-(J4-Pin_2) -> +5V
- J6 pad 1: GND -> GPIO26_ADC0_LDR
- J7 pad 2: +5V -> Net-(J7-Pin_2)
- Q3 pad 1: +3V3 -> Net-(Q3-G)
- Q3 pad 2: WS2812_RGB_LED -> GND
- Q3 pad 3: Net-(Q3-D) -> /CONNS & PERIPHERALS/BUZZER_LOW
- R1 pad 1: Net-(J1-CC1) -> Net-(R1-Pad1)
- R1 pad 2: GND -> /RP2040 & USB/~{RESET}
- R10 pad 1: +3V3 -> Net-(D2-K)
- R10 pad 2: /PAGE2/~{QSPI_CS} -> PWR_OFF_SW_N
- R11 pad 1: Net-(D3-A) -> /RP2040 & USB/~{QSPI_CS}
- R11 pad 2: +5V -> /RP2040 & USB/USBBOOT
- R12 pad 1: /PAGE2/~{QSPI_CS} -> Net-(D3-A)
- R12 pad 2: /PAGE2/USBBOOT -> +5V
- R15 pad 1: /PAGE2/~{RESET} -> Net-(D4-A)
- R15 pad 2: /PAGE2/PROG1 -> +3V3
- R16 pad 1: unconnected-(R16-Pad1) -> /RP2040 & USB/~{RESET}
- R16 pad 2: /PAGE2/PROG2 -> /RP2040 & USB/PROG1
- R16 pad 3: /PAGE2/SWDIO -> /RP2040 & USB/SWCLK
- R17 pad 1: Net-(D4-A) -> unconnected-(R17-Pad1)
- R17 pad 2: +3V3 -> /RP2040 & USB/PROG2
- R19 pad 1: +3V3 -> +5V
- R19 pad 2: BUTTON_0 -> /CONNS & PERIPHERALS/BUZZER_HIGH
- R2 pad 1: Net-(J1-CC2) -> Net-(J1-CC1)
- R20 pad 1: Net-(D5-DIN) -> +3V3
- R20 pad 2: Net-(Q3-D) -> BUTTON_0
- R21 pad 1: Net-(R21-Pad1) -> GPIO11
- R21 pad 2: BUTTON_1 -> Net-(Q3-G)
- R22 pad 1: +5V -> Net-(D5-DIN)
- R22 pad 2: Net-(Q3-D) -> Net-(Q4-D)
- R23 pad 1: +3V3 -> +5V
- R23 pad 2: BUTTON_1 -> Net-(Q4-D)
- R24 pad 1: +3V3 -> Net-(R24-Pad1)
- R24 pad 2: PPS -> BUTTON_1
- R25 pad 2: WS2812_RGB_LED -> BUTTON_1
- R26 pad 2: /PAGE3/OLED_RST -> WS2812_RGB_LED
- R27 pad 1: GPIO26_ADC0_LDR -> +3V3
- R27 pad 2: GND -> PPS
- R28 pad 1: Net-(J4-Pin_2) -> +3V3
- R28 pad 2: +3V3 -> /CONNS & PERIPHERALS/OLED_RST
- R29 pad 1: GND -> GPIO26_ADC0_LDR
- R29 pad 2: Net-(J6-Pin_26) -> GND
- R3 pad 1: Net-(R3-Pad1) -> Net-(J1-CC2)
- R3 pad 2: /PAGE2/~{RESET} -> GND
- R31 pad 1: GPIO11 -> GND
- R31 pad 2: Net-(Q5-G) -> Net-(J7-Pin_26)
- R4 pad 2: /PAGE2/~{RESET} -> /RP2040 & USB/~{RESET}
- R5 pad 2: /PAGE2/GPIO25_LED -> /RP2040 & USB/GPIO25_LED
- R6 pad 1: /PAGE2/USB_D- -> /RP2040 & USB/USB_D-
- R6 pad 2: /PAGE2/D- -> /RP2040 & USB/D-
- R7 pad 1: /PAGE2/USB_D+ -> /RP2040 & USB/USB_D+
- R7 pad 2: /PAGE2/D+ -> /RP2040 & USB/D+
- R9 pad 1: Net-(D2-K) -> +3V3
- R9 pad 2: PWR_OFF_SW_N -> /RP2040 & USB/~{QSPI_CS}
- SW1 pad 2: Net-(R3-Pad1) -> Net-(R1-Pad1)
- SW3 pad 2: /PAGE2/USBBOOT -> /RP2040 & USB/USBBOOT
- SW5 pad 2: Net-(R21-Pad1) -> Net-(R24-Pad1)
- TP3 pad 1: /PAGE2/~{RESET} -> /RP2040 & USB/~{RESET}
- TP4 pad 1: +5V -> GND
- TP5 pad 1: GND -> +5V
- TP6 pad 1: +3V3 -> GND
- TP7 pad 1: GND -> +3V3
- U1 pad 1: /PAGE2/USB_D- -> +3V3
- U1 pad 2: GND -> /RP2040 & USB/UART0_TX
- U1 pad 3: /PAGE2/USB_D+ -> /RP2040 & USB/UART0_RX
- U1 pad 4: unconnected-(U1-IO3-Pad4) -> GPIO2
- U1 pad 5: VBUS -> GPIO3
- U1 pad 6: unconnected-(U1-IO4-Pad6) -> GPIO4
- U2 pad 1: +3V3 -> /RP2040 & USB/USB_D+
- U2 pad 2: /PAGE2/UART0_TX -> GND
- U2 pad 3: /PAGE2/UART0_RX -> /RP2040 & USB/USB_D-
- U2 pad 4: GPIO2 -> unconnected-(U2-IO3-Pad4)
- U2 pad 5: GPIO3 -> VBUS
- U2 pad 6: GPIO4 -> unconnected-(U2-IO4-Pad6)
- U4 pad 1: /PAGE2/~{QSPI_CS} -> /RP2040 & USB/~{QSPI_CS}
- U4 pad 2: /PAGE2/QSPI_SD1 -> /RP2040 & USB/QSPI_SD1
- U4 pad 3: /PAGE2/QSPI_SD2 -> /RP2040 & USB/QSPI_SD2
- U4 pad 5: /PAGE2/QSPI_SD0 -> /RP2040 & USB/QSPI_SD0
- U4 pad 6: /PAGE2/QSPI_SCLK -> /RP2040 & USB/QSPI_SCLK
- U4 pad 7: /PAGE2/QSPI_SD3 -> /RP2040 & USB/QSPI_SD3
- Y1 pad 1: Net-(U2-XOUT) -> Net-(U1-XOUT)
- Y1 pad 3: Net-(U2-XIN) -> Net-(U1-XIN)
Routing:
- net /RP2040 & USB/USB_D-: track 0.00 -> 14.9 mm, vias 0 -> 1
- net /RP2040 & USB/USB_D+: track 0.00 -> 14.4 mm, vias 0 -> 1
- net Net-(J1-CC2): track 0.00 -> 5.55 mm, vias 0 -> 1
- net Net-(J1-CC1): track 0.00 -> 2.81 mm, vias 0 -> 1
- net GND: track 0.00 -> 0.80 mm, vias 0 -> 1
- net Net-(F1-Pad1): vias 0 -> 7
- added copper zone on B.Cu, net Net-(F1-Pad1)
- added copper zone on F.Cu, net Net-(F1-Pad1)
- added copper zone on F.Cu, net VBUS
Other:
- outline, holes or cut-outs redrawn

Commit message: changed all to single sided
Parts:
- J1, SW4, SW5: moved to F.Cu
- moved F1 98.8 mm to (154.9, 150.9)
- moved SW2 96.2 mm to (147.4, 116.5), turned to 90 degrees
- moved SW4 86.2 mm to (142.2, 130.0), turned to 180 degrees
- moved SW5 86.2 mm to (142.2, 137.5), turned to 180 degrees
- moved J1 86.0 mm to (146.0, 145.0)
- moved BT1 75.5 mm to (63.1, 125.0)
- moved J5 68.1 mm to (139.3, 103.7)
- moved G*** 62.2 mm to (64.6, 70.8)
- moved G*** 62.2 mm to (138.2, 43.9)
- moved G*** 62.2 mm to (59.8, 70.6)
- moved G*** 62.2 mm to (120.6, 45.7)
- moved G*** 62.2 mm to (79.3, 54.3)
- moved G*** 62.2 mm to (52.9, 48.6)
- moved G*** 62.2 mm to (99.2, 67.7)
- moved H7 15.0 mm to (132.0, 147.0)
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Routing:
- net /RP2040 & USB/USB_D-: track 14.9 -> 2.46 mm, vias 1 -> 0
- net /RP2040 & USB/USB_D+: track 14.4 -> 2.35 mm, vias 1 -> 0
- net Net-(J1-CC2): track 5.55 -> 0.00 mm, vias 1 -> 0
- net Net-(J1-CC1): track 2.81 -> 0.00 mm, vias 1 -> 0
- net GND: track 0.80 -> 0.00 mm, vias 1 -> 0
- net Net-(F1-Pad1): vias 7 -> 0

Commit message: layout work
Parts:
- removed TP2: GND, TestPoint:TestPoint_Pad_D1.0mm
- removed TP6, TP8: 5V, TestPoint:TestPoint_Pad_D1.0mm
- added C33: 1u, Capacitor_SMD:C_0402_1005Metric, F.Cu at (80.1, 146.6)
- added G***: LOGO, silk:tv, F.Cu at (85.3, 121.8)
- added G***: LOGO, silk:battery, F.Cu at (61.3, 124.9)
- SW2: renamed from SW1; footprint Button_Switch_SMD:SW_SPST_TL3342 -> stride_footprints:SW_SPST_TL3342_RT
- SW3, SW4, SW5: footprint Button_Switch_SMD:SW_SPST_TL3342 -> stride_footprints:SW_SPST_TL3342_RT
- moved R19 172.7 mm to (167.7, 91.7)
- moved Q3 162.5 mm to (168.9, 87.8)
- moved C19 150.3 mm to (156.1, 121.2)
- moved R18 149.4 mm to (155.2, 118.8)
- moved R24 131.7 mm to (154.0, 130.5)
- moved U3 121.3 mm to (132.0, 121.1), turned to 90 degrees
- moved D4 112.1 mm to (129.3, 113.9), turned to 180 degrees
- moved R10 111.6 mm to (129.7, 135.5), turned to 90 degrees
- moved R23 107.4 mm to (70.3, 157.9)
- moved R12 106.8 mm to (124.0, 143.6), turned to 90 degrees
- moved D3 103.0 mm to (125.0, 145.8), turned to 180 degrees
- moved C23 102.4 mm to (156.0, 130.5)
- moved Q2 101.7 mm to (125.0, 140.5), turned to 180 degrees
- moved R8 99.0 mm to (131.0, 135.5), turned to 90 degrees
- moved D2 98.2 mm to (126.0, 135.6)
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- renumbered SW2 to SW1
Connections:
- Q4 pad 2: WS2812_RGB_LED -> GPIO13_WS2812_RGB_LED
- R26 pad 2: WS2812_RGB_LED -> GPIO13_WS2812_RGB_LED
- U2 pad 1: /RP2040 & USB/USB_D+ -> /RP2040 & USB/USB_D-
- U2 pad 3: /RP2040 & USB/USB_D- -> /RP2040 & USB/USB_D+
Routing:
- net GND: track 0.00 -> 84.5 mm, vias 0 -> 53
- net /RP2040 & USB/USB_D+: track 2.35 -> 24.5 mm
- net /RP2040 & USB/USB_D-: track 2.46 -> 23.1 mm
- net +3V3: track 0.00 -> 19.2 mm, vias 0 -> 3
- net I2C_SDA: track 0.00 -> 17.6 mm, vias 0 -> 2
- net I2C_SCL: track 0.00 -> 13.7 mm, vias 0 -> 2
- net /RP2040 & USB/SWCLK: track 0.00 -> 12.2 mm
- net /RP2040 & USB/PROG2: track 0.00 -> 10.9 mm
- net /RP2040 & USB/~{RESET}: track 0.00 -> 10.8 mm
- net /RP2040 & USB/SWDIO: track 0.00 -> 10.6 mm
- net Net-(U1-VREG_VOUT): track 0.00 -> 9.93 mm
- net (no net): track 0.00 -> 9.30 mm, vias 0 -> 6
- net Net-(U1-XIN): track 0.00 -> 6.94 mm
- net /CONNS & PERIPHERALS/OLED_RST: track 0.00 -> 5.96 mm
- net /RP2040 & USB/QSPI_SD3: track 0.00 -> 5.93 mm
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- removed copper zone on B.Cu, net Net-(F1-Pad1)
- removed copper zone on F.Cu, net VBUS
Other:
- outline, holes or cut-outs redrawn
- board text added: "FFC EXPANSION"
- board text removed: "BUZ"
- board text removed: "FFC"
- board text removed: "PWR_SW"
