File: pcb/PAGE2.kicad_sch (KiCad schematic)
At the start: 66 parts, among them J1 USB_C_Receptacle_USB2.0, J2 PROG, Q1 AO3401A, Q2 AO3401A, SW1 SSSS811101, SW2 TS-1187A-B-A-B, SW3 TS-1187A-B-A-B, U1 RP2040, U2 SRV05-4, U3 RT9080-33GJ5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

Commit message: Ordered pcba
Parts:
- removed R12: 2.2k, Resistor_SMD:R_0402_1005Metric, symbol Device:R_Small_US
- added R21: 4.7k, Resistor_SMD:R_0402_1005Metric, symbol Device:R_Small_US
- C1: LCSC PN (none) -> C15525; LCSC Part # C15525 -> (none); lcsc C15525 -> (none)
- C10, C11, C14, C15, C3, C4, C5, C6, C7, C9: LCSC PN (none) -> C1525; LCSC Part # C1525 -> (none); lcsc C1525 -> (none)
- C12, C13: LCSC PN (none) -> C32949; LCSC Part # C32949 -> (none); lcsc C32949 -> (none)
- C16, C17: LCSC PN (none) -> C23733; LCSC Part # C23733 -> (none); lcsc C23733 -> (none)
- C18, C2, C8: LCSC PN (none) -> C52923; LCSC Part # C52923 -> (none); lcsc C52923 -> (none)
- D1: value LED -> LED_Y; footprint LED_SMD:LED_0603_1608Metric -> LED_SMD:LED_0805_2012Metric; LCSC PN (none) -> C2296; LCSC Part # C72038 -> (none); desc VFtyp 2V, VFmax 2.3V, Yellow -> (none); lcsc C72038 -> (none)
- D2: LCSC PN (none) -> C8062; LCSC Part # C8062 -> (none); lcsc C8062 -> (none)
- D3: value LED -> LED_G; footprint LED_SMD:LED_0603_1608Metric -> LED_SMD:LED_0805_2012Metric; Color BLU -> GRN; LCSC PN (none) -> C2297; LCSC Part # C72041 -> (none); desc VFtyp 2.8V, VFmax 3.1V, Blue -> (none); lcsc C72041 -> (none)
- D4: value LED -> LED_G; footprint LED_SMD:LED_0603_1608Metric -> LED_SMD:LED_0805_2012Metric; LCSC PN (none) -> C2297; LCSC Part # C72043 -> (none); desc VFtyp 3.3V, VFmax 3.7V, Green -> (none); lcsc C72043 -> (none)
- F1: LCSC PN (none) -> C516068; LCSC Part # C516068 -> (none); lcsc C516068 -> (none)
- FID1, FID2, H1, H2, H3, H4, H5, H6, H7, TP1, TP3, TP5, TP7: now left out of the parts list
- J1: LCSC PN (none) -> C167321; LCSC Part # C167321 -> (none); lcsc C167321 -> (none)
- J2: now fitted; now left out of the parts list
- Q1, Q2: LCSC PN (none) -> C15127; LCSC Part # C15127 -> (none); lcsc C15127 -> (none)
- R1, R11: LCSC PN (none) -> C11702; LCSC Part # C11702 -> (none); lcsc C11702 -> (none)
- R10, R8: LCSC PN (none) -> C25741; LCSC Part # C25741 -> (none); lcsc C25741 -> (none)
- R13, R14: LCSC PN (none) -> C25900; LCSC Part # C25900 -> (none); lcsc C25900 -> (none)
- R15: value 300 -> 1k; LCSC PN (none) -> C11702; LCSC Part # C25102 -> (none); lcsc C25102 -> (none)
- R16, R17: LCSC PN (none) -> C17168; LCSC Part # C17168 -> (none); lcsc C17168 -> (none)
- R2: LCSC PN (none) -> C25905; LCSC Part # C25744 -> (none); desc (none) -> C25905; lcsc C25744 -> (none)
- R3: LCSC PN (none) -> C25905; LCSC Part # C25744 -> (none); lcsc C25744 -> (none)
- R4, R9: LCSC PN (none) -> C25744; LCSC Part # C25744 -> (none); lcsc C25744 -> (none)
- R5: LCSC PN (none) -> C25879; LCSC Part # C25879 -> (none); lcsc C25879 -> (none)
- R6, R7: LCSC PN (none) -> C25092; LCSC Part # C25092 -> (none); lcsc C25092 -> (none)
- SW1: LCSC PN (none) -> C109335; LCSC Part # C109335 -> (none); lcsc C109335 -> (none)
- SW2, SW3: LCSC PN (none) -> C318884; LCSC Part # C318884 -> (none); lcsc C318884 -> (none)
- TP4: LCSC PN (none) -> C5199799; LCSC Part # C5199799 -> (none); lcsc C5199799 -> (none); now left out of the parts list
- U1: LCSC PN (none) -> C2040; LCSC Part # C2040 -> (none); lcsc C2040 -> (none)
- U2: LCSC PN (none) -> C85364; LCSC Part # C85364 -> (none); lcsc C85364 -> (none)
- U3: LCSC PN (none) -> C841192; LCSC Part # C841192 -> (none); lcsc C841192 -> (none)
- U4: LCSC PN (none) -> C2940195; LCSC Part # C2940195 -> (none); lcsc C2940195 -> (none)
- Y1: LCSC PN (none) -> C9002; LCSC Part # C9002 -> (none); lcsc C9002 -> (none)
Connections:
- net +5V: now also R21.2
- net at D3.2 (A): now also R21.1
Other:
- moved on the sheet: D4
