File: pcb/PAGE3.kicad_sch (KiCad schematic)
At the start: 43 parts, among them J3 FFC 24, J4 5V, J5 5V, J6 5V, J7 OLED, Q3 AO3400A, Q4 2N7002, SW4 TS-1187A-B-A-B, SW5 TS-1187A-B-A-B, U5 DS1307Z+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

Commit message: Ordered pcba
Parts:
- BT1: LCSC PN (none) -> C70377; LCSC Part # C70377 -> (none); lcsc C70377 -> (none)
- C19, C23, C25, C32: LCSC PN (none) -> C1525; LCSC Part # C1525 -> (none); lcsc C1525 -> (none)
- C20, C21, C24, C26, C27, C29, C30, C33: LCSC PN (none) -> C52923; LCSC Part # C52923 -> (none); lcsc C52923 -> (none)
- C22: LCSC PN (none) -> C15525; LCSC Part # C15525 -> (none); lcsc C15525 -> (none)
- C28: LCSC PN (none) -> C12530; LCSC Part # C12530 -> (none); lcsc C12530 -> (none)
- C31: LCSC PN (none) -> C23733; LCSC Part # C23733 -> (none); lcsc C23733 -> (none)
- D5: LCSC PN (none) -> C965555; LCSC Part # C965555 -> (none); lcsc C965555 -> (none)
- D6: LCSC PN (none) -> C2480; LCSC Part # C2480 -> (none); lcsc C2480 -> (none)
- J3: LCSC PN (none) -> C202112; LCSC Part # C202112 -> (none); lcsc C202112 -> (none)
- J4, J5, J6: LCSC PN (none) -> C160402; LCSC Part # C160402 -> (none); lcsc C160402 -> (none)
- J7: LCSC PN (none) -> C2890596; LCSC Part # C2890596 -> (none); lcsc C2890596 -> (none)
- Q3: LCSC PN (none) -> C20917; LCSC Part # C20917 -> (none); lcsc C20917 -> (none)
- Q4: LCSC PN (none) -> C8545; LCSC Part # C8545 -> (none); lcsc C8545 -> (none)
- R18, R19, R24, R30: LCSC PN (none) -> C11702; LCSC Part # C11702 -> (none); lcsc C11702 -> (none)
- R20, R23, R25, R26, R27, R28, R29: LCSC PN (none) -> C25744; LCSC Part # C25744 -> (none); lcsc C25744 -> (none)
- R22: LCSC PN (none) -> C25125; LCSC Part # C25125 -> (none); lcsc C25125 -> (none)
- R31: LCSC PN (none) -> C25778; LCSC Part # C25778 -> (none); lcsc C25778 -> (none)
- SW4, SW5: LCSC PN (none) -> C318884; LCSC Part # C318884 -> (none); lcsc C318884 -> (none)
- U5: LCSC PN (none) -> C8959; LCSC Part # C8959 -> (none); lcsc C8959 -> (none)
- Y2: LCSC PN (none) -> C95361; LCSC Part # C95361 -> (none); lcsc C95361 -> (none)
Other:
- note added: "49.9 C25120 used"
