File: pcb/clock_pcb.kicad_pcb (KiCad board)
At the start: 2 copper layers, 100 x 50 mm, 116 parts, among them J1 USB_C_Receptacle_USB2.0, J2 PROG, J3 FFC 24, J4 5V, J5 5V, J6 5V, J7 OLED, Q1 AO3401A, Q2 AO3401A, Q3 AO3400A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

Commit message: Ordered pcba
Parts:
- removed R12: 2.2k, Resistor_SMD:R_0402_1005Metric
- added R21: 4.7k, Resistor_SMD:R_0402_1005Metric, F.Cu at (125.4, 140.9)
- added kibuzzard-68226165: G***, kibuzzard-68226165, F.Cu at (84.1, 101.1)
- added kibuzzard-68226193: G***, kibuzzard-68226193, F.Cu at (61.4, 125.4)
- added kibuzzard-682261A9: G***, kibuzzard-682261A9, F.Cu at (86.0, 139.8)
- added kibuzzard-682261BD: G***, kibuzzard-682261BD, F.Cu at (107.2, 101.2)
- added kibuzzard-682261D0: G***, kibuzzard-682261D0, F.Cu at (100.8, 101.2)
- added kibuzzard-682261E0: G***, kibuzzard-682261E0, F.Cu at (114.7, 101.1)
- added kibuzzard-682261F1: G***, kibuzzard-682261F1, F.Cu at (110.9, 122.2)
- added kibuzzard-68226263: G***, kibuzzard-68226263, F.Cu at (105.8, 148.4)
- D1: value LED -> LED_Y; footprint LED_SMD:LED_0603_1608Metric -> LED_SMD:LED_0805_2012Metric
- D3, D4: value LED -> LED_G; footprint LED_SMD:LED_0603_1608Metric -> LED_SMD:LED_0805_2012Metric
- R15: value 300 -> 1k
- moved D4 0.50 mm to (136.4, 116.9)
Routing:
- net GND: track 149.7 -> 150.2 mm
Other:
- board text removed: "FFC EXPANSION"
- board text removed: "HUMMINGBIRD V1.0"
- board text removed: "LDR"
- board text removed: "PWR"
- board text removed: "SWITCH"
