File: pcb/v2/CONNS.kicad_sch (KiCad schematic)
At the start: 43 parts, among them J1 LDR, J10 SW, J12 OLED, J2 PWR, J8 FFC 24, Q5 AO3400A, Q6 2N7002, SW6 TS-1187A-B-A-B, SW7 TS-1187A-B-A-B, U6 DS1307Z+, Y3 32.768kHz

Commit message: started v2
Parts:
- removed Y3: 32.768kHz, Crystal:Crystal_SMD_3215-2Pin_3.2x1.5mm, symbol Device:Crystal_Small
- added R27: GL5516, OptoDevice:R_LDR_5.1x4.3mm_P3.4mm_Vertical, symbol Sensor_Optical:LDR07
- added U5: DS1302ZN+, Package_SO:SOIC-8_3.9x4.9mm_P1.27mm, symbol Timer_RTC:DS1302ZN+
- added Y2: 32.768kHz, Crystal:Crystal_SMD_3215-2Pin_3.2x1.5mm, symbol Device:Crystal_Small
- renumbered BT2 to BT1, BZ2 to BZ1, C43 to C21, C48 to C22, C35 to C23, C34 to C24, C38 to C25, C36 to C26, C37 to C27, C39 to C28, C40 to C29, C41 to C30, C42 to C31, C44 to C32, C45 to C33, C46 to C34, C47 to C35, D8 to D6, J8 to J3, J2 to J4, J10 to J5, J1 to J6, J12 to J7, Q5 to Q6, Q6 to Q7, R41 to R25, R42 to R26, R12 to R28, R32 to R29, R39 to R30, R36 to R31, R37 to R32, R38 to R36, R40 to R37, R43 to R38, SW6 to SW4, SW7 to SW5
Connections:
- net at U6.1 (X1): now also Y2.2
- net at U6.2 (X2): now also Y2.1
Other:
- note added: "CAN THIS BE BETWEEN THE FETS to make switch work?"
- note added: "OLED LCSC PN: C2890596 Wisevision N096-2864KSWEG01-H30 Controller SSD1306"
- note added: "Senba Sensing Tech GL5516 C125626 200KΩ (dark) to 10KΩ (10 lux brightness) LDR 5kΩ~10kΩ to 500kΩ THT Dark 150mV - 400mV Typ - 1.6V Light Sim meeeeeeeeeeeeeeeeeeeeeeee"
- moved on the sheet: BT1, C23, C27, D7, Q7, R30, R34, R35, R36, U6

Commit message: schematic pick
Parts:
- removed BZ1: CMT-8504-100-SMT-TR, Buzzer_Beeper:MagneticBuzzer_CUI_CMT-8504-100-SMT, symbol stride_symbols:Buzzer_CMT-8504-100-SMT-TR
- removed Q7: 2N7002, Package_TO_SOT_SMD:SOT-23, symbol Transistor_FET:2N7002
- removed R35, R36: 10k, Resistor_SMD:R_0402_1005Metric, symbol Device:R_Small_US
- removed U5: DS1302ZN+, Package_SO:SOIC-8_3.9x4.9mm_P1.27mm, symbol Timer_RTC:DS1302ZN+
- added C32, C34, C35, C36, C37: 1u, Capacitor_SMD:C_0402_1005Metric, symbol Device:C_Small
- added C41: 0.1u, Capacitor_SMD:C_0402_1005Metric, symbol Device:C_Small
- added D6, D8, D9: WS2812B-2020, StrideLibrary:WS2812B-2020, symbol LED_Extra:WS2812B-2020
- added J8: LDR, Connector_JST:JST_SH_SM02B-SRSS-TB_1x02-1MP_P1.00mm_Horizontal, symbol Connector_Generic:Conn_01x02
- added R29, R30: 0, Resistor_SMD:R_0402_1005Metric, symbol Device:R_Small_US
- added R38: 1k, Resistor_SMD:R_0402_1005Metric, symbol Device:R_Small_US
- added R40: 10k, Resistor_SMD:R_0402_1005Metric, symbol Device:R_Small_US
- added U6: SN74LVC1T45DBV, Package_TO_SOT_SMD:SOT-23-6, symbol Logic_LevelTranslator:SN74LVC1T45DBV
- D7: footprint stride_footprints:WS2812B-2020 -> StrideLibrary:WS2812B-2020
- R34: value 51 -> 49.9; LCSC PN C25125 -> C25120
- R39: renamed from R27; now fitted
- U5: renamed from U6; LCSC PN (none) -> C26858
- renumbered C24 to C21, C25 to C22, C33 to C23, C34 to C24, C28 to C25, C29 to C26, C31 to C27, C23 to C28, C30 to C29, C32 to C30, C35 to C31, C27 to C33, C21 to C38, C26 to C39, C22 to C40, D6 to D10, J7 to J4, J4 to J5, J5 to J6, J6 to J7, R29 to R25, R32 to R26, R28 to R27, R31 to R28, R37 to R31, R30 to R32, R38 to R33, R26 to R35, R25 to R36, R33 to R37
Connections:
- net +3V3: now also C35.1, R38.2, U6.6 (VCCB); no longer C28.1, U5.8 (VCC)
- net +5V: now also C28.1, U5.8 (VCC), C32.1, C34.1, C36.1, C37.1, D6.4 (VDD), D8.4 (VDD), D9.4 (VDD), J8.2 (Pin_2), U6.1 (VCCA); no longer J5.2 (Pin_2)
- net BUZZER_LOW: now also J8.1 (Pin_1)
- net GND: now also C32.2, C34.2, C35.2, C36.2, C37.2, C41.2, D6.2 (VSS), D8.2 (VSS), D9.2 (VSS), J8.MP (Mounting_Point), R40.2, U6.2 (GND), U6.5 (DIR)
- net GPIO12_PPS: no longer J3.7 (Pin_7)
- net GPIO13_WS2812_RGB_LED: now also U6.4 (B)
- net WS2812_DOUT: now also D8.1 (DOUT); no longer D7.1 (DOUT)
- net at R34.2: now also U6.3 (A)
- net at J3.1 (Pin_1): now also R29.1
- net at R39.1: now also R38.1
- net GPIO27_ADC1_LDR: now reaches R39.2
- net GPIO27_ADC1_LDR: now also C41.1, R40.1
- net BUTTON_0 renamed GPIO14_BUTTON_0
- net BUTTON_1 renamed GPIO15_BUTTON_1
- net GPIO26_ADC0_LDR renamed GPIO26_ADC0_LDR_EXT
- net GPIO27_ADC1 renamed GPIO18
- new net: D6.3 (DIN), D7.1 (DOUT)
- new net: D8.3 (DIN), D9.1 (DOUT)
- new net: J3.7 (Pin_7), R30.1
- new net DOUT: D6.1 (DOUT), D9.3 (DIN)
- new net UNFUSED_VBUS: J5.2 (Pin_2)
- no-connect marks 2 -> 3
Other:
- note added: "011 110A R/W 011 1101 R/W = 0x3C"
- note added: "110 1000 R/W = 0x68"
- note added: "Allows external switch to control the boards power if PCB switch is off."
- note added: "Hirose_FFC 24: Pitch 0.5mm, FFC Tck 0.3mm Pins connect on PCB side FFC SAME 24P 0.5mm 12CM - C36268 3cm C5248005 FFC OPP. 24P 0.5mm 12CM - C24318 3cm C5248014"
- note added: "OLED Wisevision N096-2864KSWEG01-H30 LCSC PN: C2890596 Controller SSD1306"
- note added: "PU at Pi"
- note added: "Senba Sensing Tech GL5516 C125626 500kΩ (dark) to 5kΩ~10kΩ (10 lux brightness)"
- note added: "Vil=2.2V, works for 3v3 IO"
- note removed: "49.9 C25120 used"
- note removed: "CAN THIS BE BETWEEN THE FETS to make switch work?"
- note removed: "D/CP (ADDR): 0111100b' GND 0x3C <- 0111101b' VDD 0x3D"
- note removed: "Hirose_FFC 24: FFC SAME C36268 FFC OPP. C24318"
- note removed: "LDR: 1528-2141-ND 200KΩ (dark) to 10KΩ (10 lux brightness) Dark 150mV - 400mV Typ - 1.6V Light"
- note removed: "OLED LCSC PN: C2890596 Wisevision N096-2864KSWEG01-H30 Controller SSD1306"
- note removed: "Senba Sensing Tech GL5516 C125626 200KΩ (dark) to 10KΩ (10 lux brightness) LDR 5kΩ~10kΩ to 500kΩ THT Dark 150mV - 400mV Typ - 1.6V Light Sim meeeeeeeeeeeeeeeeeeeeeeee"
- note removed: "logic lvl shifter"
- moved on the sheet: BT1, C21, C22, C28, C33, C39, D10, D7, J3, Q6, R25, R26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
