File: pcb/v2/RP2040.kicad_sch (KiCad schematic)
At the start: 67 parts, among them J13 USB_C_Receptacle_USB2.0, J14 PROG, Q1 AO3400A, Q2 AO3400A, Q3 AO3400A, Q7 AO3401A, Q8 AO3401A, SW10 TS-1187A-B-A-B, SW8 TS-1187A-B-A-B, SW9 SSSS811101, U10 W25Q64JV, U7 SRV05-4, U8 RP2040, U9 RT9080-33GJ5, Y4 XYDBPCNANF-12MHZ

Commit message: started v2
Parts:
- removed C65: 4.7u, Capacitor_SMD:C_0402_1005Metric, symbol Device:C_Small
- removed SW10, SW8: TS-1187A-B-A-B, stride_footprints:SW_SPST_TL3342_RT, symbol Switch:SW_Push
- removed U9: RT9080-33GJ5, Package_TO_SOT_SMD:SOT-23-5, symbol Regulator_Linear:AP2112K-3.3
- added C17, C20: 4.7u, Capacitor_SMD:C_0402_1005Metric, symbol Device:C_Small
- added C19: 10u, Capacitor_SMD:C_0402_1005Metric, symbol Device:C_Small
- added SW1, SW2: TS-1187A-B-A-B, Button_Switch_SMD:SW_SPST_TS-1088-xR020, symbol Switch:SW_Push
- added U4: AMS1117-3.3, Package_TO_SOT_SMD:SOT-223-3_TabPin2, symbol Regulator_Linear:AMS1117-3.3
- SW3: renamed from SW9; footprint stride_footprints:SSSS811101 -> StrideLibrary:SSSS811101
- U1: renamed from U8; footprint stride_footprints:QFN-56_EP_7x7_Pitch0.4mm -> StrideLibrary:QFN-56_EP_7x7_Pitch0.4mm
- renumbered C49 to C1, C58 to C10, C59 to C11, C60 to C12, C61 to C13, C62 to C14, C63 to C15, C66 to C16, C64 to C18, C50 to C2, C51 to C3, C52 to C4, C53 to C5, C54 to C6, C55 to C7, C56 to C8, C57 to C9, D2 to D1, D9 to D2, D10 to D3, D1 to D4, D4 to D5, F2 to F1, J13 to J1, J14 to J2, Q7 to Q3, Q8 to Q4, Q3 to Q5, R45 to R1, R50 to R10, R5 to R11, R52 to R12, R54 to R13, R48 to R14, R56 to R15, R57 to R16, R51 to R17, R53 to R18, R8 to R19, R46 to R2, R59 to R20, R60 to R21, R6 to R22, R7 to R23, R10 to R24, R44 to R3, R1 to R4, R2 to R5, R47 to R6, R4 to R7, R3 to R8, R49 to R9, TP6 to TP3, TP9 to TP4, TP10 to TP5, U7 to U2, U10 to U3, Y4 to Y1
Connections:
- net +3V3: now also C19.1, C20.1, U4.2 (VO)
- net +5V: now also C17.1, U4.3 (VI)
- net GND: now also C17.2, C19.2, C20.2, SW1.2, SW2.1, U4.1 (GND)
- net USBBOOT: now also SW2.2
- net at R3.1: now also SW1.1
- net test: now reaches J1.A5 (CC1), R1.1
Other:
- note added: "1A Max"
- note removed: "600mA Max"
- moved on the sheet: C18, D2, D5, Q5, R14, R22, R23, R24, TP5, U2

Commit message: schematic pick
Parts:
- renumbered C17 to C1, C7 to C10, C9 to C11, C11 to C12, C15 to C13, C16 to C14, C8 to C15, C10 to C16, C14 to C17, C5 to C18, C12 to C19, C18 to C2, C13 to C20, C19 to C3, C20 to C4, C1 to C5, C2 to C6, C3 to C7, C4 to C8, C6 to C9, D3 to D1, D5 to D2, D1 to D3, D2 to D5, Q3 to Q1, Q4 to Q2, Q5 to Q3, Q1 to Q4, Q2 to Q5, R18 to R10, R23 to R11, R5 to R12, R8 to R13, R12 to R14, R13 to R15, R6 to R16, R3 to R17, R9 to R18, R10 to R19, R24 to R2, R16 to R20, R15 to R21, R20 to R22, R21 to R23, R14 to R24, R2 to R3, R7 to R4, R11 to R5, R19 to R6, R4 to R7, R22 to R8, R17 to R9, SW3 to SW1, SW1 to SW3, TP5 to TP3, TP3 to TP5, U4 to U1, U1 to U3, U3 to U4
Connections:
- net UNFUSED_VBUS: now reaches F1.2, J1.A4 (VBUS), J1.A9 (VBUS), J1.B4 (VBUS), J1.B9 (VBUS)
- net GPIO26_ADC0_LDR renamed GPIO26_ADC0_LDR_EXT
- net GPIO27_ADC1 renamed GPIO27_ADC1_LDR
Other:
- moved on the sheet: F1, TP2
