File: pcb/v2/clock_module_v2.0.kicad_pcb (KiCad board)
At the start: 4 copper layers, 110 parts, among them J1 LDR, J10 SW, J2 PWR, J8 FFC 24, Q1 AO3400A, Q2 AO3400A, Q3 AO3400A, Q5 AO3400A, Q6 2N7002, Q7 AO3401A, Q8 AO3401A, SW1 TS-1187A-B-A-B, SW2 TS-1187A-B-A-B, SW9 SSSS811101, U1 DS1302ZN+, U10 W25Q64JV, U2 AMS1117-3.3, U6 DS1307Z+, U7 SRV05-4, U8 RP2040, Y1 32.768kHz, Y4 XYDBPCNANF-12MHZ

Commit message: schematic pick
Parts:
- removed BZ2: CMT-8504-100-SMT-TR, Buzzer_Beeper:MagneticBuzzer_CUI_CMT-8504-100-SMT
- removed H12, H13, H14: Mounting_Hole, MountingHole:MountingHole_2.7mm_M2.5
- removed the Q6 at (128.4, 63.0)
- removed the R38 at (146.8, 64.2)
- removed the U1 at (138.2, 50.8)
- added C36: 0.1u, Capacitor_SMD:C_0402_1005Metric, F.Cu at (117.8, 39.2)
- added C37: 1u, Capacitor_SMD:C_0402_1005Metric, F.Cu at (114.4, 53.0)
- added C38: 1u, Capacitor_SMD:C_0402_1005Metric, F.Cu at (114.4, 55.0)
- added C39: 1u, Capacitor_SMD:C_0402_1005Metric, F.Cu at (114.4, 56.9)
- added C40: 1u, Capacitor_SMD:C_0402_1005Metric, F.Cu at (114.4, 58.9)
- added C41: 1u, Capacitor_SMD:C_0402_1005Metric, F.Cu at (114.4, 60.9)
- added D7: WS2812B-2020, StrideLibrary:WS2812B-2020, F.Cu at (117.8, 56.5)
- added H1: Tooling_Hole_JLC, MountingHole:ToolingHole_1.152mm, F.Cu at (44.5, 114.0)
- added H2: Tooling_Hole_JLC, MountingHole:ToolingHole_1.152mm, F.Cu at (44.5, 116.5)
- added H3: Tooling_Hole_JLC, MountingHole:ToolingHole_1.152mm, F.Cu at (44.5, 119.0)
- added H5: Mounting_Hole, MountingHole:MountingHole_2.7mm_M2.5_DIN965_Pad_TopBottom, F.Cu at (40.1, 122.2)
- added H6: Mounting_Hole, MountingHole:MountingHole_2.7mm_M2.5_DIN965_Pad_TopBottom, F.Cu at (40.1, 128.4)
- added H7: Mounting_Hole, MountingHole:MountingHole_2.7mm_M2.5_DIN965_Pad_TopBottom, F.Cu at (40.1, 134.7)
- added J8: LDR, Connector_JST:JST_SH_SM02B-SRSS-TB_1x02-1MP_P1.00mm_Horizontal, F.Cu at (129.4, 28.5)
- added R27: GL5516, OptoDevice:R_LDR_5.1x4.3mm_P3.4mm_Vertical, F.Cu at (120.9, 35.2)
- added R39: 10k, Resistor_SMD:R_0402_1005Metric, F.Cu at (106.9, 39.3)
- added R40: 1k, Resistor_SMD:R_0402_1005Metric, F.Cu at (106.9, 41.3)
- added U5: SN74LVC1T45DBV, Package_TO_SOT_SMD:SOT-23-6, F.Cu at (118.4, 52.5)
- H4: renamed from H11; footprint MountingHole:MountingHole_2.7mm_M2.5 -> MountingHole:MountingHole_2.7mm_M2.5_DIN965_Pad_TopBottom
- R34: value 51 -> 49.9
- R35: value 10k -> 0
- moved FID1 119.7 mm to (45.0, 122.0)
- moved FID2 119.7 mm to (45.0, 125.5)
- moved H4 116.5 mm to (40.1, 116.0)
- moved SW3 110.4 mm to (79.0, 26.5)
- moved TP5 110.3 mm to (37.3, 36.0)
- moved D1 109.5 mm to (54.2, 24.0)
- moved F1 107.2 mm to (44.2, 51.9)
- moved C18 106.4 mm to (47.0, 29.1)
- moved U2 104.0 mm to (44.0, 55.9)
- moved U3 102.1 mm to (38.4, 92.7)
- moved U4 101.5 mm to (40.7, 30.3)
- moved C17 97.9 mm to (47.0, 27.1)
- moved C19 96.9 mm to (47.0, 31.0)
- moved D5 96.2 mm to (54.9, 34.2)
- moved C16 96.1 mm to (45.3, 79.4)
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- renumbered C49 to C1, C58 to C10, C59 to C11, C60 to C12, C61 to C13, C62 to C14, C63 to C15, C66 to C16, C2 to C17, C64 to C18, C3 to C19, C50 to C2, C1 to C20, C43 to C21, C48 to C22, C35 to C23, C34 to C24, C38 to C25, C36 to C26, C37 to C27, C39 to C28, C40 to C29, C51 to C3, C41 to C30, C42 to C31, C44 to C32, C45 to C33, C46 to C34, C47 to C35, C52 to C4, C53 to C5, C54 to C6, C55 to C7, C56 to C8, C57 to C9, D2 to D1, D9 to D2, D10 to D3, D1 to D4, D4 to D5, D8 to D6, F2 to F1, FID3 to FID1, FID4 to FID2, J8 to J3, J2 to J4, J10 to J5, J1 to J6, Q7 to Q3, Q8 to Q4, Q3 to Q5, Q5 to Q6, R45 to R1, R50 to R10, R5 to R11, R52 to R12, R54 to R13, R48 to R14, R56 to R15, R57 to R16, R51 to R17, R53 to R18, R8 to R19, R46 to R2, R6 to R22, R7 to R23, R10 to R24, R41 to R25, R42 to R26, R12 to R28, R32 to R29, R44 to R3, R39 to R30, R36 to R31, R37 to R32, R40 to R37, R43 to R38, R1 to R4, R2 to R5, R47 to R6, R4 to R7, R3 to R8, R49 to R9, SW2 to SW1, SW1 to SW2, SW9 to SW3, TP6 to TP3, TP9 to TP4, TP10 to TP5, U8 to U1, U7 to U2, U10 to U3, U2 to U4, Y4 to Y1, Y1 to Y2
Connections:
- net GPIO26_ADC0_LDR renamed GPIO26_ADC0_LDR_EXT
- C23 pad 1: +3V3 -> +5V
- C24 pad 1: BUTTON_0 -> GPIO14_BUTTON_0
- C25 pad 1: BUTTON_1 -> GPIO15_BUTTON_1
- F1 pad 2: Net-(F2-Pad2) -> UNFUSED_VBUS
- J3 pad 19: GPIO27_ADC1 -> GPIO18
- J3 pad 7: GPIO12_PPS -> Net-(J3-Pin_7)
- J4 pad 2: +5V -> UNFUSED_VBUS
- R28 pad 2: BUTTON_0 -> GPIO14_BUTTON_0
- R29 pad 2: BUTTON_0 -> GPIO14_BUTTON_0
- R31 pad 2: BUTTON_1 -> GPIO15_BUTTON_1
- R32 pad 2: BUTTON_1 -> GPIO15_BUTTON_1
- R34 pad 2: Net-(Q6-D) -> Net-(U5-A)
- R35 pad 1: +5V -> Net-(J3-Pin_7)
- R35 pad 2: Net-(Q6-D) -> unconnected-(R35-Pad2)
- U1 pad 39: GPIO27_ADC1 -> GPIO27_ADC1_LDR
- U6 pad 8: +3V3 -> +5V
Other:
- board text added: "3V3"
- board text added: "5V"
- board text added: "BOOT"
- board text added: "HUMMINGBIRD V2.0"
- board text added: "LDR PWR SW BUZZER"
- board text added: "OFF"
- board text added: "ON"
- board text added: "PBAD"
- board text added: "RST"
- board text added: "VBUS"
- board text removed: "Check my hole vs jlc tooling hole"
