File: pcb/v2/clock_module_v2.0.kicad_sch (KiCad schematic)
At the start: 10 parts

Commit message: started v2
Parts:
- TP1: renamed from TP8; LCSC Status (none) -> Extended; now not fitted
- renumbered FID3 to FID1, FID4 to FID2, H8 to H1, H9 to H2, H10 to H3, H11 to H4, H12 to H5, H13 to H6, H14 to H7
Changed lines of the file:
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@@
 		(dnp no)
 		(fields_autoplaced yes)
-		(property "Reference" "H8"
+		(property "Reference" "H1"
 			(at 320.04 230.2315 0)
 			(effects
@@
 			(project "clock_module_v2.0"
 				(path "/e9b4505e-6f30-405f-a63f-0ff05fc75bc0"
-					(reference "H8")
+					(reference "H1")
 					(unit 1)
 				)
@@
 		(dnp no)
 		(fields_autoplaced yes)
-		(property "Reference" "H14"
+		(property "Reference" "H7"
 			(at 360.68 236.064 0)
 			(effects
@@
 			(project "clock_module_v2.0"
 				(path "/e9b4505e-6f30-405f-a63f-0ff05fc75bc0"
-					(reference "H14")
+					(reference "H7")
 					(unit 1)
 				)
@@
 		(in_bom no)
 		(on_board yes)
-		(dnp no)
-		(property "Reference" "TP8"
+		(dnp yes)
+		(property "Reference" "TP1"
 			(at 372.745 228.6 90)
 			(effects
@@
 			)
 		)
+		(property "LCSC Status" "Extended"
+			(at 376.555 231.14 90)
+			(effects
+				(font
+					(size 1.27 1.27)
+				)
+				(hide yes)
+			)
+		)
 		(pin "1"
 		)
@@
 			(project "clock_module_v2.0"
 				(path "/e9b4505e-6f30-405f-a63f-0ff05fc75bc0"
-					(reference "TP8")
+					(reference "TP1")
 					(unit 1)
 				)
@@
 		(on_board yes)
 		(dnp no)
-		(property "Reference" "H11"
+		(property "Reference" "H4"
 			(at 352.425 231.775 0)
 			(effects
@@
 			(project "clock_module_v2.0"
 				(path "/e9b4505e-6f30-405f-a63f-0ff05fc75bc0"
-					(reference "H11")
+					(reference "H4")
 					(unit 1)
 				)
@@
 		(dnp no)
 		(fields_autoplaced yes)
-		(property "Reference" "H13"
+		(property "Reference" "H6"
 			(at 360.68 231.619 0)
 			(effects
@@
 			(project "clock_module_v2.0"
 				(path "/e9b4505e-6f30-405f-a63f-0ff05fc75bc0"
-					(reference "H13")
+					(reference "H6")
 					(unit 1)
 				)
@@
 		(dnp no)
 		(fields_autoplaced yes)
-		(property "Reference" "FID3"
+		(property "Reference" "FID1"
 			(at 338.709 230.2315 0)
 			(effects
@@
 			(project "clock_module_v2.0"
 				(path "/e9b4505e-6f30-405f-a63f-0ff05fc75bc0"
-					(reference "FID3")
+					(reference "FID1")
 					(unit 1)
 				)
@@
 		(dnp no)
 		(fields_autoplaced yes)
-		(property "Reference" "H12"
+		(property "Reference" "H5"
 			(at 352.425 236.064 0)
 			(effects
@@
 			(project "clock_module_v2.0"
 				(path "/e9b4505e-6f30-405f-a63f-0ff05fc75bc0"
-					(reference "H12")
+					(reference "H5")
 					(unit 1)
 				)
@@
 		(dnp no)
 		(fields_autoplaced yes)
-		(property "Reference" "H10"
+		(property "Reference" "H3"
 			(at 327.66 230.2315 0)
 			(effects
@@
 			(project "clock_module_v2.0"
 				(path "/e9b4505e-6f30-405f-a63f-0ff05fc75bc0"
-					(reference "H10")
+					(reference "H3")
 					(unit 1)
 				)
@@
 		(dnp no)
 		(fields_autoplaced yes)
-		(property "Reference" "H9"
+		(property "Reference" "H2"
 			(at 320.04 234.6765 0)
 			(effects
@@
 			(project "clock_module_v2.0"
 				(path "/e9b4505e-6f30-405f-a63f-0ff05fc75bc0"
-					(reference "H9")
+					(reference "H2")
 					(unit 1)
 				)
@@
 		(dnp no)
 		(fields_autoplaced yes)
-		(property "Reference" "FID4"
+		(property "Reference" "FID2"
 			(at 338.709 234.6765 0)
 			(effects
@@
 			(project "clock_module_v2.0"
 				(path "/e9b4505e-6f30-405f-a63f-0ff05fc75bc0"
-					(reference "FID4")
+					(reference "FID2")
 					(unit 1)
 				)
@@
 		(on_board yes)
 		(dnp no)
-		(property "Reference" "#PWR0138"
+		(property "Reference" "#PWR01"
 			(at 382.27 239.395 0)
 			(effects
@@
 			(project "clock_module_v2.0"
 				(path "/e9b4505e-6f30-405f-a63f-0ff05fc75bc0"
-					(reference "#PWR0138")
-					(unit 1)
-				)
+					(reference "#PWR01")
+					(unit 1)
+				)

Commit message: schematic pick
Parts:
- removed H3: Tooling_Hole_JLC, stride_footprints:JLC_Tooling_Hole, symbol Mechanical:MountingHole
- added H4: Mounting_Hole, MountingHole:MountingHole_2.7mm_M2.5_DIN965_Pad_TopBottom, symbol Mechanical:MountingHole
- H1, H2: footprint stride_footprints:JLC_Tooling_Hole -> MountingHole:ToolingHole_1.152mm
- H3: renamed from H4; footprint MountingHole:MountingHole_2.7mm_M2.5 -> MountingHole:MountingHole_2.7mm_M2.5_DIN965_Pad_TopBottom
- H5: value Mounting_Hole -> Tooling_Hole_JLC; footprint MountingHole:MountingHole_2.7mm_M2.5 -> MountingHole:ToolingHole_1.152mm
- H6, H7: footprint MountingHole:MountingHole_2.7mm_M2.5 -> MountingHole:MountingHole_2.7mm_M2.5_DIN965_Pad_TopBottom
Other:
- moved on the sheet: H3
